File: breadboarder.brd (EAGLE design)
At the start: 100 x 80 mm, 13 parts, among them IC1 AVR-MEGA8-PPTH, Q1 MOSFET-NCHANNEL2N7000

Commit message: think I've got all of breadboarder parts down
...but who knows.
Parts:
- removed R1: (no value), SparkFun-Passives:1206
- added AGND, AVCC: M02PTH, SparkFun-Connectors:1X02
- added D2, D3, D4, D5, D6, D7, D8: Yellow, SparkFun-LED:LED-1206
- added S1, S2: (no value), SparkFun-Electromechanical:TACTILE-PTH
Connections:
- removed net LED: R1.1
- removed net N$14: D1.A, R1.2
- new net N$2: D2.C, R2.P$8
- new net N$3: D3.C, R2.P$7
- new net N$4: D4.C, R2.P$6
- new net N$5: D5.C, R2.P$5
- new net N$6: D6.C, R2.P$4
- new net N$7: D7.C, R2.P$3
- new net N$8: D8.C, R2.P$2
- new net N$9: D1.C, R2.P$9
- new net PB0: BANKB.8, D1.A, IC1.14
- new net PB1: BANKB.7, D2.A, IC1.15
- new net PB2: BANKB.6, D3.A, IC1.16
- new net PB3: BANKB.5, D4.A, IC1.17, ISP.4
- new net PB4: BANKB.4, D5.A, IC1.18, ISP.1
- new net PB5: BANKB.3, D6.A, IC1.19, ISP.3
- new net PB6: BANKB.2, D7.A, IC1.9
- new net PB7: BANKB.1, D8.A, IC1.10
- new net PC0: BANKC.7, IC1.23
- new net PC1: BANKC.6, IC1.24
- new net PC2: BANKC.5, IC1.25
- new net PC3: BANKC.4, IC1.26
- new net PC4: BANKC.3, IC1.27
- new net PC5: BANKC.2, IC1.28
- new net PD0: BANKD.8, FTDI.TXO, IC1.2
- new net PD1: BANKD.7, FTDI.RXI, IC1.3
- new net PD2: BANKD.6, IC1.4, S2.1
- new net PD3: BANKD.5, IC1.5
- new net PD4: BANKD.4, IC1.6
- new net PD5: BANKD.3, IC1.11
- new net PD6: BANKD.2, IC1.12
- new net PD7: BANKD.1, IC1.13
- net AGND: now also AGND.2, IC1.22
- net AREF: now also IC1.21
- net AVCC: now also AVCC.1
- net GND: now also AGND.1, FTDI.GND, IC1.8, ISP.6, S1.4, S2.4; no longer D1.C
- net RESET: now also BANKC.1, IC1.1, ISP.5, S1.1
- net VCC: now also AVCC.2, FTDI.VCC, IC1.7, ISP.2

Commit message: lol.  first try = sucessful autoroute
now comes the process of refinement...
Parts:
- removed C3: 0.1uF, rcl:C1206
- removed D1, D2, D3, D4, D5, D6, D7, D8: Yellow, SparkFun-LED:LED-1206
- removed S1, S2: (no value), SparkFun-Electromechanical:TACTILE-PTH
- added BUTTON, RESET: (no value), SparkFun-Electromechanical:TACTILE-PTH
- added C1: 0.1uF, SparkFun-Capacitors:CAP-PTH-SMALL-KIT
- added LED1, LED2, LED3, LED4, LED5, LED6, LED7, LED8, LED9: (no value), SparkFun-LED:LED3MM
- added R1: 1k Ohm, SparkFun-Passives:AXIAL-0.3
- moved AGND 165.4 mm to (61.0, 33.0), turned to 180 degrees
- moved AVCC 158.7 mm to (61.0, 30.5), turned to 180 degrees
- moved Q1 123.7 mm to (68.6, 34.3), turned to 90 degrees
- moved R2 123.1 mm to (72.4, 35.6), turned to 90 degrees
- moved ANALOG 104.7 mm to (58.4, 25.4)
- moved POWER 53.4 mm to (24.1, 2.54), turned to 180 degrees
- moved BANKD 17.8 mm to (68.6, 2.54), turned to 180 degrees
- moved FTDI 12.0 mm to (33.0, 36.8)
Connections:
- new net N$10: LED9.K, R1.P$2
- net GND: now also BUTTON.4, C1.2, R1.P$1, RESET.4; no longer C3.2, S1.4, S2.4
- net N$2: now also LED1.K, R2.P$9; no longer D2.C, R2.P$8
- net N$3: now also LED2.K, R2.P$8; no longer D3.C, R2.P$7
- net N$4: now also LED3.K, R2.P$7; no longer D4.C, R2.P$6
- net N$5: now also LED4.K, R2.P$6; no longer D5.C, R2.P$5
- net N$6: now also LED5.K, R2.P$5; no longer D6.C, R2.P$4
- net N$7: now also LED6.K, R2.P$4; no longer D7.C, R2.P$3
- net N$8: now also LED7.K, R2.P$3; no longer D8.C, R2.P$2
- net N$9: now also LED8.K, R2.P$2; no longer D1.C, R2.P$9
- net PB0: now also LED1.A; no longer D1.A
- net PB1: now also LED2.A; no longer D2.A
- net PB2: now also LED3.A; no longer D3.A
- net PB3: now also LED4.A; no longer D4.A
- net PB4: now also LED5.A; no longer D5.A
- net PB5: now also LED6.A; no longer D6.A
- net PB6: now also LED7.A; no longer D7.A
- net PB7: now also LED8.A; no longer D8.A
- net PD2: now also BUTTON.1; no longer S2.1
- net RESET: now also RESET.1; no longer S1.1
- net VCC: now also C1.1, LED9.A; no longer C3.1
Routing:
- net GND: track 0.00 -> 146.7 mm
- net PB4: track 0.00 -> 114.8 mm
- net RESET: track 0.00 -> 111.4 mm
- net PB5: track 0.00 -> 109.9 mm
- net VCC: track 0.00 -> 97.8 mm
- net PB3: track 0.00 -> 92.4 mm
- net PD0: track 0.00 -> 81.2 mm
- net PB6: track 0.00 -> 58.7 mm
- net PC1: track 0.00 -> 50.7 mm
- net PD1: track 0.00 -> 50.0 mm
- net PB0: track 0.00 -> 47.0 mm
- net PB1: track 0.00 -> 43.1 mm
- net PB2: track 0.00 -> 43.1 mm
- net PC0: track 0.00 -> 39.5 mm
- net PD2: track 0.00 -> 37.1 mm
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- added copper zone on layer 16, net GND
- added copper zone on layer 1, net VCC
Other:
- board size 100 x 80 mm -> 101.3 x 81.3 mm
