File: breadboarder.sch (EAGLE design)
At the start: 13 parts, among them IC1 AVR-MEGA8-PPTH, Q1 MOSFET-NCHANNEL2N7000

Commit message: think I've got all of breadboarder parts down
...but who knows.
Parts:
- removed R1: (no value), SparkFun-Passives:RESISTOR1206
- added AGND, AVCC: M02PTH, SparkFun-Connectors:M02PTH
- added D2, D3, D4, D5, D6, D7, D8: Yellow, SparkFun-LED:LED-YELLOWLILYPAD
- added S1, S2: (no value), SparkFun-Electromechanical:TAC_SWITCHPTH
Connections:
- removed net LED: R1.1
- removed net N$14: D1.A, R1.2
- new net N$2: D2.C, R2.8
- new net N$3: D3.C, R2.7
- new net N$4: D4.C, R2.6
- new net N$5: D5.C, R2.5
- new net N$6: D6.C, R2.4
- new net N$7: D7.C, R2.3
- new net N$8: D8.C, R2.2
- new net N$9: D1.C, R2.9
- new net PB0: BANKB.8, D1.A, IC1.PB0(ICP)
- new net PB1: BANKB.7, D2.A, IC1.PB1(OC1A)
- new net PB2: BANKB.6, D3.A, IC1.PB2(SS/OC1B)
- new net PB3: BANKB.5, D4.A, IC1.PB3(MOSI/OC2), ISP.4
- new net PB4: BANKB.4, D5.A, IC1.PB4(MISO), ISP.1
- new net PB5: BANKB.3, D6.A, IC1.PB5(SCK), ISP.3
- new net PB6: BANKB.2, D7.A, IC1.PB6(XTAL1/TOSC1)
- new net PB7: BANKB.1, D8.A, IC1.PB7(XTAL2/TOSC2)
- new net PC0: BANKC.7, IC1.PC0(ADC0)
- new net PC1: BANKC.6, IC1.PC1(ADC1)
- new net PC2: BANKC.5, IC1.PC2(ADC2)
- new net PC3: BANKC.4, IC1.PC3(ADC3)
- new net PC4: BANKC.3, IC1.PC4(ADC4/SDA)
- new net PC5: BANKC.2, IC1.PC5(ADC5/SCL)
- new net PD0: BANKD.8, FTDI.3, IC1.PD0(RXD)
- new net PD1: BANKD.7, FTDI.2, IC1.PD1(TXD)
- new net PD2: BANKD.6, IC1.PD2(INT0), S2.1
- new net PD3: BANKD.5, IC1.PD3(INT1)
- new net PD4: BANKD.4, IC1.PD4(XCK/T0)
- new net PD5: BANKD.3, IC1.PD5(T1)
- new net PD6: BANKD.2, IC1.PD6(AIN0)
- new net PD7: BANKD.1, IC1.PD7(AIN1)
- net AGND: now also AGND.2, IC1.AGND
- net AREF: now also IC1.AREF
- net AVCC: now also AVCC.1
- net GND: now also AGND.1, FTDI.6, IC1.GND@1, ISP.6, S1.4, S2.4; no longer D1.C
- net RESET: now also BANKC.1, IC1.PC6(/RESET), ISP.5, S1.1
- net VCC: now also AVCC.2, FTDI.4, IC1.VCC@1, ISP.2
Other:
- moved on the sheet: D1, FTDI

Commit message: lol.  first try = sucessful autoroute
now comes the process of refinement...
Parts:
- removed C3: 0.1uF, rcl:C-EUC1206
- removed D1, D2, D3, D4, D5, D6, D7, D8: Yellow, SparkFun-LED:LED-YELLOWLILYPAD
- added C1: 0.1uF, SparkFun-Capacitors:CAPKIT
- added LED1, LED2, LED3, LED4, LED5, LED6, LED7, LED8, LED9: (no value), SparkFun-LED:LED3MM
- added R1: 1k Ohm, SparkFun-Passives:RESISTORAXIAL-0.3
- renumbered S1 to RESET, S2 to BUTTON
Connections:
- new net N$10: LED9.C, R1.2
- net GND: now also C1.2, R1.1; no longer C3.2
- net N$2: now also LED1.C, R2.9; no longer D2.C, R2.8
- net N$3: now also LED2.C, R2.8; no longer D3.C, R2.7
- net N$4: now also LED3.C, R2.7; no longer D4.C, R2.6
- net N$5: now also LED4.C, R2.6; no longer D5.C, R2.5
- net N$6: now also LED5.C, R2.5; no longer D6.C, R2.4
- net N$7: now also LED6.C, R2.4; no longer D7.C, R2.3
- net N$8: now also LED7.C, R2.3; no longer D8.C, R2.2
- net N$9: now also LED8.C, R2.2; no longer D1.C, R2.9
- net PB0: now also LED1.A; no longer D1.A
- net PB1: now also LED2.A; no longer D2.A
- net PB2: now also LED3.A; no longer D3.A
- net PB3: now also LED4.A; no longer D4.A
- net PB4: now also LED5.A; no longer D5.A
- net PB5: now also LED6.A; no longer D6.A
- net PB6: now also LED7.A; no longer D7.A
- net PB7: now also LED8.A; no longer D8.A
- net VCC: now also C1.1, LED9.A; no longer C3.1
