File: mega_simplest_classboard_redux.sch (EAGLE design)
At the start: 9 parts, among them IC1 MEGA8-P

Commit message: tested version minimal classboard
is it a minimal classboard or a mega breadboarder?
8-LED breakout untested, mostly-symmetric design
Parts:
- removed FTDISERIAL: (no value), pinhead:PINHD-1X6
- added AREF, RESET: (no value), pinhead:PINHD-1X1
- added FTDI: (no value), SparkFun-Connectors:M06SIP
- PORTB: value B -> (none); device pinhead:PINHD-1X8 -> SparkFun-Connectors:M081X08
- PORTC: value C -> (none); device pinhead:PINHD-1X6 -> SparkFun-Connectors:M06SIP
- PORTD: value D -> (none); device pinhead:PINHD-1X8 -> SparkFun-Connectors:M081X08
- POWER: value (none) -> M02PTH; device pinhead:PINHD-1X2 -> SparkFun-Connectors:M02PTH
Connections:
- removed net N$2: IC1.PC6(/RESET), ISP.5
- new net AREF: AREF.1, IC1.AREF
- new net RESET: IC1.PC6(/RESET), ISP.5, RESET.1
- net GND: now also FTDI.6, POWER.1; no longer FTDISERIAL.1, POWER.2
- net PORTB0: now also PORTB.8; no longer PORTB.1
- net PORTB1: now also PORTB.7; no longer PORTB.2
- net PORTB2: now also PORTB.6; no longer PORTB.3
- net PORTB3: now also PORTB.5; no longer PORTB.4
- net PORTB4: now also PORTB.4; no longer PORTB.5
- net PORTB5: now also PORTB.3; no longer PORTB.6
- net PORTB6: now also PORTB.2; no longer PORTB.7
- net PORTB7: now also PORTB.1; no longer PORTB.8
- net PORTC0: now also PORTC.6; no longer PORTC.1
- net PORTC1: now also PORTC.5; no longer PORTC.2
- net PORTC2: now also PORTC.4; no longer PORTC.3
- net PORTC3: now also PORTC.3; no longer PORTC.4
- net PORTC4: now also PORTC.2; no longer PORTC.5
- net PORTC5: now also PORTC.1; no longer PORTC.6
- net PORTD0: now also FTDI.3, PORTD.8; no longer FTDISERIAL.4, PORTD.1
- net PORTD1: now also FTDI.2, PORTD.7; no longer FTDISERIAL.5, PORTD.2
- net PORTD2: now also PORTD.6; no longer PORTD.3
- net PORTD3: now also PORTD.5; no longer PORTD.4
- net PORTD4: now also PORTD.4; no longer PORTD.5
- net PORTD5: now also PORTD.3; no longer PORTD.6
- net PORTD6: now also PORTD.2; no longer PORTD.7
- net PORTD7: now also PORTD.1; no longer PORTD.8
- net VCC: now also FTDI.4, POWER.2; no longer FTDISERIAL.3, POWER.1
Other:
- moved on the sheet: POWER
